Commit message: added color to mount and tool, added visual to the gazebo environment

File: abb_irb120_gazebo/urdf/irb120_surgical_macro.xacro (robot description, xacro)
@@ -126,4 +126,65 @@
     <turnGravityOff>true</turnGravityOff>
   </gazebo>
+  <!-- change the color of different links of the robot -->
+  <gazebo reference="${prefix}mount_1">
+    <visual>
+      <material>
+        <script>
+          <uri>file://media/materials/scripts/gazebo.material</uri>
+          <name>Gazebo/Grey</name>
+        </script>
+      </material>
+    </visual>
+  </gazebo>
+  <gazebo reference="${prefix}mount_2">
+    <visual>
+      <material>
+        <script>
+          <uri>file://media/materials/scripts/gazebo.material</uri>
+          <name>Gazebo/Grey</name>
+        </script>
+      </material>
+    </visual>
+  </gazebo>
+  <gazebo reference="${prefix}mount_3">
+    <visual>
+      <material>
+        <script>
+          <uri>file://media/materials/scripts/gazebo.material</uri>
+          <name>Gazebo/Grey</name>
+        </script>
+      </material>
+    </visual>
+  </gazebo>
+  <gazebo reference="${prefix}plate_1">
+    <visual>
+      <material>
+        <script>
+          <uri>file://media/materials/scripts/gazebo.material</uri>
+          <name>Gazebo/RedTransparentOverlay</name>
+        </script>
+      </material>
+    </visual>
+  </gazebo>
+  <gazebo reference="${prefix}plate_2">
+    <visual>
+      <material>
+        <script>
+          <uri>file://media/materials/scripts/gazebo.material</uri>
+          <name>Gazebo/Green</name>
+        </script>
+      </material>
+    </visual>
+  </gazebo>
+  <gazebo reference="${prefix}link_7">
+    <visual>
+      <material>
+        <script>
+          <uri>file://media/materials/scripts/gazebo.material</uri>
+          <name>Gazebo/Black</name>
+        </script>
+      </material>
+    </visual>
+  </gazebo>
   <!-- ros_control plugin -->
   <gazebo>

File: abb_irb120_support/urdf/irb120_surgical_macro.xacro (robot description, xacro)
@@ -1,11 +1,26 @@
 <?xml version="1.0"?>
 <robot xmlns:xacro="http://ros.org/wiki/xacro">
+  <!-- include all the dependent xacros -->
   <xacro:include filename="$(find abb_resources)/urdf/common_materials.xacro"/>
   <xacro:include filename="$(find abb_irb120_support)/urdf/mount_macro.xacro"/>
   <xacro:include filename="$(find abb_irb120_support)/urdf/surgical_tool_macro.xacro"/>
+  <xacro:include filename="$(find abb_irb120_support)/urdf/plate_macro.xacro"/>
+  <!-- give parameters to the dependent xacros -->
+  <!-- prefix = name of your robot -->
+  <!-- parent = parent link of the part "the link where the part will be attached" -->
   <xacro:mount prefix=""/>
   <xacro:mount_joints prefix="" parent="tool0"/>
   <xacro:surgical_tool prefix=""/>
   <xacro:surgical_tool_joints prefix="" parent="mount_3"/>
+  <!-- plate = imaginary area to show RCM movement -->
+  <!-- dimensions of the plate -->
+  <!-- size = dimensions of the plate -->
+  <!-- hole = radius of the hole in plate -->
+  <xacro:plate prefix="" size="0.1 0.1 0.001" hole="0.02"/>
+  <!-- plate_joints = where the plate is attached wrt to the Robot -->
+  <!-- we attach it to main base_link which is fixed -->
+  <!-- origin_xyz = change the position of the center of plate -->
+  <!-- origin_rpy = change the orientation of the plate -->
+  <xacro:plate_joints prefix="" parent="base_link" origin_xyz="0.4 0 0.35" origin_rpy="0 0 0"/>
   <xacro:macro name="abb_irb120_surgical" params="prefix">
     <!-- link list -->

Commit message: changed to position controller

File: abb_irb120_gazebo/urdf/irb120_surgical_macro.xacro (robot description, xacro)
@@ -9,5 +9,5 @@
     <type>transmission_interface/SimpleTransmission</type>
     <joint name="${prefix}joint_1">
-      <hardwareInterface>PositionJointInterface</hardwareInterface>
+      <hardwareInterface>EffortJointInterface</hardwareInterface>
     </joint>
     <actuator name="${prefix}motor1">
@@ -18,5 +18,5 @@
     <type>transmission_interface/SimpleTransmission</type>
     <joint name="${prefix}joint_2">
-      <hardwareInterface>PositionJointInterface</hardwareInterface>
+      <hardwareInterface>EffortJointInterface</hardwareInterface>
     </joint>
     <actuator name="${prefix}motor2">
@@ -27,5 +27,5 @@
     <type>transmission_interface/SimpleTransmission</type>
     <joint name="${prefix}joint_3">
-      <hardwareInterface>PositionJointInterface</hardwareInterface>
+      <hardwareInterface>EffortJointInterface</hardwareInterface>
     </joint>
     <actuator name="${prefix}motor3">
@@ -36,5 +36,5 @@
     <type>transmission_interface/SimpleTransmission</type>
     <joint name="${prefix}joint_4">
-      <hardwareInterface>PositionJointInterface</hardwareInterface>
+      <hardwareInterface>EffortJointInterface</hardwareInterface>
     </joint>
     <actuator name="${prefix}motor4">
@@ -45,5 +45,5 @@
     <type>transmission_interface/SimpleTransmission</type>
     <joint name="${prefix}joint_5">
-      <hardwareInterface>PositionJointInterface</hardwareInterface>
+      <hardwareInterface>EffortJointInterface</hardwareInterface>
     </joint>
     <actuator name="${prefix}motor5">
@@ -54,5 +54,5 @@
     <type>transmission_interface/SimpleTransmission</type>
     <joint name="${prefix}joint_6">
-      <hardwareInterface>PositionJointInterface</hardwareInterface>
+      <hardwareInterface>EffortJointInterface</hardwareInterface>
     </joint>
     <actuator name="${prefix}motor6">
@@ -63,5 +63,5 @@
     <type>transmission_interface/SimpleTransmission</type>
     <joint name="${prefix}joint_7">
-      <hardwareInterface>PositionJointInterface</hardwareInterface>
+      <hardwareInterface>EffortJointInterface</hardwareInterface>
     </joint>
     <actuator name="${prefix}motor7">
@@ -72,5 +72,5 @@
     <type>transmission_interface/SimpleTransmission</type>
     <joint name="${prefix}joint_8">
-      <hardwareInterface>PositionJointInterface</hardwareInterface>
+      <hardwareInterface>EffortJointInterface</hardwareInterface>
     </joint>
     <actuator name="${prefix}motor8">
@@ -81,5 +81,5 @@
     <type>transmission_interface/SimpleTransmission</type>
     <joint name="${prefix}joint_9">
-      <hardwareInterface>PositionJointInterface</hardwareInterface>
+      <hardwareInterface>EffortJointInterface</hardwareInterface>
     </joint>
     <actuator name="${prefix}motor9">
@@ -90,5 +90,5 @@
     <type>transmission_interface/SimpleTransmission</type>
     <joint name="${prefix}joint_a">
-      <hardwareInterface>PositionJointInterface</hardwareInterface>
+      <hardwareInterface>EffortJointInterface</hardwareInterface>
     </joint>
     <actuator name="${prefix}motora">

File: abb_irb120_support/urdf/irb120_surgical_macro.xacro (robot description, xacro)
@@ -179,5 +179,5 @@
       <parent link="${prefix}base_link"/>
       <child link="${prefix}link_1"/>
-      <limit effort="0" lower="-2.87979" upper="2.87979" velocity="4.36332"/>
+      <limit effort="100.0" lower="-2.87979" upper="2.87979" velocity="4.36332"/>
       <axis xyz="0 0 1"/>
       <dynamics damping="0.0" friction="0.0"/>
@@ -187,5 +187,5 @@
       <parent link="${prefix}link_1"/>
       <child link="${prefix}link_2"/>
-      <limit effort="0" lower="-1.91986" upper="1.91986" velocity="4.36332"/>
+      <limit effort="100.0" lower="-1.91986" upper="1.91986" velocity="4.36332"/>
       <axis xyz="0 1 0"/>
       <dynamics damping="0.0" friction="0.0"/>
@@ -195,5 +195,5 @@
       <parent link="${prefix}link_2"/>
       <child link="${prefix}link_3"/>
-      <limit effort="0" lower="-1.91986" upper="1.22173" velocity="4.36332"/>
+      <limit effort="100.0" lower="-1.91986" upper="1.22173" velocity="4.36332"/>
       <axis xyz="0 1 0"/>
       <dynamics damping="0.0" friction="0.0"/>
@@ -203,5 +203,5 @@
       <parent link="${prefix}link_3"/>
       <child link="${prefix}link_4"/>
-      <limit effort="0" lower="-2.79253" upper="2.79253" velocity="5.58505"/>
+      <limit effort="100.0" lower="-2.79253" upper="2.79253" velocity="5.58505"/>
       <axis xyz="1 0 0"/>
       <dynamics damping="0.0" friction="0.0"/>
@@ -211,5 +211,5 @@
       <parent link="${prefix}link_4"/>
       <child link="${prefix}link_5"/>
-      <limit effort="0" lower="-2.094395" upper="2.094395" velocity="5.58505"/>
+      <limit effort="100.0" lower="-2.094395" upper="2.094395" velocity="5.58505"/>
       <axis xyz="0 1 0"/>
       <dynamics damping="0.0" friction="0.0"/>
@@ -219,5 +219,5 @@
       <parent link="${prefix}link_5"/>
       <child link="${prefix}link_6"/>
-      <limit effort="0" lower="-6.98132" upper="6.98132" velocity="7.33038"/>
+      <limit effort="100.0" lower="-6.98132" upper="6.98132" velocity="7.33038"/>
       <axis xyz="1 0 0"/>
       <dynamics damping="0.0" friction="0.0"/>
