Commit message: changed the ralative position of the tool

File: abb_irb120_support/urdf/irb120_3_58_macro.xacro (robot description, xacro)
@@ -161,36 +161,36 @@
       </inertial>
       <visual>
+        <origin xyz="0 0 0" rpy="0 0 3.1415926"/>
+        <geometry>
+          <mesh filename="package://dvrk_model/PSM/meshes/main_insertion_Link.STL"/>
+        </geometry>
+        <xacro:material_abb_black />
+      </visual>
+      <collision>
+        <origin xyz="0 0 0" rpy="0 0 3.1415926"/>
+        <geometry>
+          <mesh filename="package://dvrk_model/PSM/meshes/main_insertion_Link.STL"/>
+        </geometry>
+        <xacro:material_abb_yellow />
+      </collision>
+    </link>
+    <link name="${prefix}link_8">
+      <inertial>
+        <mass value="0.137"/>
+        <origin xyz="-1.1311E-08 -7.4559E-09 -0.0058234" rpy="0 0 3.1415926"/>
+        <inertia ixx="0.001" ixy="0" ixz="0" iyy="0.001" iyz="0" izz="0.001"/>
+      </inertial>
+      <visual>
+        <origin xyz="0 0 0" rpy="0 0 3.1415926"/>
+        <geometry>
+          <mesh filename="package://dvrk_model/PSM/meshes/tool_roll_link.STL"/>
+        </geometry>
+        <xacro:material_abb_black />
+      </visual>
+      <collision>
         <origin xyz="0 0 0" rpy="0 0 3.14159"/>
         <geometry>
-          <mesh filename="package://dvrk_model/PSM/meshes/main_insertion_Link.STL"/>
-        </geometry>
-        <xacro:material_abb_black />
-      </visual>
-      <collision>
-        <origin xyz="0 0 0" rpy="0 0 3.14159"/>
-        <geometry>
-          <mesh filename="package://dvrk_model/PSM/meshes/main_insertion_Link.STL"/>
-        </geometry>
-        <xacro:material_abb_yellow />
-      </collision>
-    </link>
-    <link name="${prefix}link_8">
-      <inertial>
-        <mass value="0.137"/>
-        <origin xyz="-1.1311E-08 -7.4559E-09 -0.0058234" rpy="0 0 3.14159"/>
-        <inertia ixx="0.001" ixy="0" ixz="0" iyy="0.001" iyz="0" izz="0.001"/>
-      </inertial>
-      <visual>
-        <origin xyz="0 0 0" rpy="0 0 3.14159"/>
-        <geometry>
           <mesh filename="package://dvrk_model/PSM/meshes/tool_roll_link.STL"/>
         </geometry>
-        <xacro:material_abb_black />
-      </visual>
-      <collision>
-        <origin xyz="0 0 0" rpy="0 0 3.14159"/>
-        <geometry>
-          <mesh filename="package://dvrk_model/PSM/meshes/tool_roll_link.STL"/>
-        </geometry>
         <xacro:material_abb_yellow />
       </collision>
@@ -199,9 +199,9 @@
       <inertial>
         <mass value="0.137"/>
-        <origin xyz="0.0035766 -4.8675E-05 4.4413E-06" rpy="0 0 3.14159"/>
-        <inertia ixx="0.001" ixy="0" ixz="0" iyy="0.001" iyz="0" izz="0.001"/>
-      </inertial>
-      <visual>
-        <origin xyz="0 0 0" rpy="0 0 3.14159"/>
+        <origin xyz="0.0035766 -4.8675E-05 4.4413E-06" rpy="0 0 3.1415926"/>
+        <inertia ixx="0.001" ixy="0" ixz="0" iyy="0.001" iyz="0" izz="0.001"/>
+      </inertial>
+      <visual>
+        <origin xyz="0 0 0" rpy="0 0 3.1415926"/>
         <geometry>
           <mesh filename="package://dvrk_model/PSM/meshes/tool_pitch_link.STL"/>
@@ -210,5 +210,5 @@
       </visual>
       <collision>
-        <origin xyz="0 0 0" rpy="0 0 3.14159"/>
+        <origin xyz="0 0 0" rpy="0 0 3.1415926"/>
         <geometry>
           <mesh filename="package://dvrk_model/PSM/meshes/tool_pitch_link.STL"/>
@@ -318,5 +318,5 @@
       <parent link="${prefix}link_6"/>
       <child link="${prefix}link_7"/>
-      <origin xyz="0.1 0 0" rpy="3.1415926 0 0" />
+      <origin xyz="0.1 0 0.1" rpy="3.1415926 -1.5707963267949 0" />
     </joint>
     <joint name="${prefix}joint_7" type="revolute">

Commit message: changed the distance of tool wrt ABB e-eff

File: abb_irb120_support/urdf/irb120_3_58_macro.xacro (robot description, xacro)
@@ -318,5 +318,5 @@
       <parent link="${prefix}link_6"/>
       <child link="${prefix}link_7"/>
-      <origin xyz="0.1 0 0.1" rpy="3.1415926 -1.5707963267949 0" />
+      <origin xyz="0.051 0 0.1" rpy="3.1415926 -1.5707963267949 0" />
     </joint>
     <joint name="${prefix}joint_7" type="revolute">

File: abb_irb120_support/urdf/mount_macro.xacro (robot description, xacro)
@@ -56,5 +56,5 @@
         <origin xyz="0 0 0" rpy="0 0 0"/>
         <geometry>
-          <box size="0.05 0.08 0.12"/>
+          <box size="0.05 0.08 0.1"/>
         </geometry>
         <material name="blue">
@@ -65,5 +65,5 @@
         <origin xyz="0 0 0" rpy="0 0 0"/>
         <geometry>
-          <box size="0.05 0.08 0.12"/>
+          <box size="0.05 0.08 0.1"/>
         </geometry>
       </collision>
@@ -85,5 +85,5 @@
       <parent link="${prefix}mount_2"/>
       <child link="${prefix}mount_3"/>
-      <origin xyz="0.015 0 0.055" rpy="0 0 0" />
+      <origin xyz="0.015 0 0.046" rpy="0 0 0" />
     </joint>
   </xacro:macro>
