Commit message: changed the weight of the mount and tool

File: abb_irb120_support/urdf/mount_macro.xacro (robot description, xacro)
@@ -5,5 +5,5 @@
     <link name="${prefix}mount_1">
       <inertial>
-        <mass value="0.050"/>
+        <mass value="0.05"/>
         <origin xyz="0 0 0" rpy="0 0 0"/>
         <inertia ixx="0.0001" ixy="0" ixz="0" iyy="0.0001" iyz="0" izz="0.0001"/>
@@ -27,5 +27,5 @@
     <link name="${prefix}mount_2">
       <inertial>
-        <mass value="0.1"/>
+        <mass value="0.05"/>
         <origin xyz="0 0 0" rpy="0 0 0"/>
         <inertia ixx="0.0001" ixy="0" ixz="0" iyy="0.0001" iyz="0" izz="0.0001"/>
@@ -49,5 +49,5 @@
     <link name="${prefix}mount_3">
       <inertial>
-        <mass value="0.1"/>
+        <mass value="0.15"/>
         <origin xyz="0 0 0" rpy="0 0 0"/>
         <inertia ixx="0.0001" ixy="0" ixz="0" iyy="0.0001" iyz="0" izz="0.0001"/>

File: abb_irb120_support/urdf/plate_macro.xacro (robot description, xacro)
@@ -4,5 +4,5 @@
     <link name="${prefix}plate_1">
       <inertial>
-        <mass value="0.1"/>
+        <mass value="0.000001"/>
         <origin xyz="0 0 0" rpy="0 0 0"/>
         <inertia ixx="0.0001" ixy="0" ixz="0" iyy="0.0001" iyz="0" izz="0.0001"/>
@@ -20,5 +20,5 @@
     <link name="${prefix}plate_2">
       <inertial>
-        <mass value="0.050"/>
+        <mass value="0.000001"/>
         <origin xyz="0 0 0" rpy="0 0 0"/>
         <inertia ixx="0.0001" ixy="0" ixz="0" iyy="0.0001" iyz="0" izz="0.0001"/>

File: abb_irb120_support/urdf/surgical_tool_macro.xacro (robot description, xacro)
@@ -5,5 +5,5 @@
     <link name="${prefix}link_7">
       <inertial>
-        <mass value="0.137"/>
+        <mass value="0.150"/>
         <origin xyz="0.0040563 -0.00010934 0.010292" rpy="0 0 0"/>
         <inertia ixx="0.001" ixy="0" ixz="0" iyy="0.001" iyz="0" izz="0.001"/>
@@ -26,5 +26,5 @@
     <link name="${prefix}link_8">
       <inertial>
-        <mass value="0.137"/>
+        <mass value="0.005"/>
         <origin xyz="-1.1311E-08 -7.4559E-09 -0.0058234" rpy="0 0 3.1415926"/>
         <inertia ixx="0.001" ixy="0" ixz="0" iyy="0.001" iyz="0" izz="0.001"/>
@@ -47,5 +47,5 @@
     <link name="${prefix}link_9">
       <inertial>
-        <mass value="0.137"/>
+        <mass value="0.005"/>
         <origin xyz="0.0035766 -4.8675E-05 4.4413E-06" rpy="0 0 3.1415926"/>
         <inertia ixx="0.001" ixy="0" ixz="0" iyy="0.001" iyz="0" izz="0.001"/>
@@ -68,5 +68,5 @@
     <link name="${prefix}link_10">
       <inertial>
-        <mass value="0.137"/>
+        <mass value="0.005"/>
         <origin xyz="0.00018874 0.0013526 -0.00091695" rpy="0 0 0" />
         <inertia ixx="0.001" ixy="0" ixz="0" iyy="0.001" iyz="0" izz="0.001"/>
@@ -89,5 +89,5 @@
     <link name="${prefix}link_11">
       <inertial>
-        <mass value="0.137"/>
+        <mass value="0.005"/>
         <origin xyz="0.00018874 0.0013526 -0.00091695" rpy="0 0 0" />
         <inertia ixx="0.001" ixy="0" ixz="0" iyy="0.001" iyz="0" izz="0.001"/>
